File: blueprints/pcb/11111.kicad_pcb (KiCad board)
At the start: 2 copper layers, 301.3 x 112 mm, 131 parts, among them J1 TRRS_MJ-4PP-9, J2 TRRS_MJ-4PP-9, SW1 SW_Push, SW10 SW_Push, SW11 SW_Push, SW12 SW_Push, SW13 SW_Push, SW14 SW_Push, SW15 SW_Push, SW16 SW_Push, SW17 SW_Push, SW18 SW_Push, SW19 SW_Push, SW2 SW_Push, SW20 SW_Push, SW21 SW_Push, SW22 SW_Push, SW23 SW_Push, SW24 SW_Push, SW25 SW_Push, SW26 SW_Push, SW27 SW_Push, SW28 SW_Push, SW29 SW_Push, SW3 SW_Push, SW30 SW_Push, SW31 SW_Push, SW32 SW_Push, SW33 SW_Push, SW34 SW_Push, SW35 SW_Push, SW36 SW_Push, SW37 SW_Push, SW38 SW_Push, SW39 SW_Push, SW4 SW_Push, SW40 SW_Push, SW41 SW_Push, SW42 SW_Push, SW43 SW_Push, SW44 SW_Push, SW45 SW_Push, SW46 SW_Push, SW47 SW_Push, SW48 SW_Push, SW49 SW_Push, SW5 SW_Push, SW50 SW_Push, SW51 SW_Push, SW52 SW_Push, SW53 SW_Push, SW54 SW_Push, SW55 SW_Push, SW56 SW_Push, SW57 SW_Push, SW58 SW_Push, SW59 SW_Push, SW6 SW_Push, SW60 SW_Push, SW61 SW_Push, SW62 SW_Push, SW7 SW_Push, SW8 SW_Push, SW9 SW_Push, U1 Pico, U2 Pico

Commit message: add 2 switches
Parts:
- removed R1, R2: 5.1k, Resistor_THT:R_Axial_DIN0204_L3.6mm_D1.6mm_P5.08mm_Vertical
- removed U3: ~, keyboard_parts:USB_type-C_dip_module_AE-USB2.0-TYPE-C
- added D57: 1N4148W, Salicylic-acid3_kbd_Parts:Diode_SMD, F.Cu at (104.3, 121.9)
- added D64: 1N4148W, Salicylic-acid3_kbd_Parts:Diode_SMD, F.Cu at (268.2, 121.9)
- added REF**: m3_Spacer_Hole_hex, keyboard_parts:m3_Spacer_Hole_hex, F.Cu at (198.9, 28.1)
- added REF**: m3_Spacer_Hole_hex, keyboard_parts:m3_Spacer_Hole_hex, F.Cu at (55.9, 88.3)
- added REF**: m3_Spacer_Hole_hex, keyboard_parts:m3_Spacer_Hole_hex, F.Cu at (276.9, 129.1)
- added REF**: m3_Spacer_Hole_hex, keyboard_parts:m3_Spacer_Hole_hex, F.Cu at (315.0, 88.2)
- added REF**: m3_Spacer_Hole_hex, keyboard_parts:m3_Spacer_Hole_hex, F.Cu at (38.5, 28.2)
- added REF**: m3_Spacer_Hole_hex, keyboard_parts:m3_Spacer_Hole_hex, F.Cu at (94.0, 129.1)
- added REF**: m3_Spacer_Hole_hex, keyboard_parts:m3_Spacer_Hole_hex, F.Cu at (332.4, 28.2)
- added REF**: USB_type-C_dip_module_AE-USB2.0-TYPE-C, keyboard_parts:USB_type-C_dip_module_AE-USB2.0-TYPE-C, F.Cu at (124.5, 23.0)
- added REF**: m3_Spacer_Hole_hex, keyboard_parts:m3_Spacer_Hole_hex, F.Cu at (172.0, 129.1)
- added REF**: m3_Spacer_Hole_hex, keyboard_parts:m3_Spacer_Hole_hex, F.Cu at (172.0, 28.2)
- added REF**: m3_Spacer_Hole_hex, keyboard_parts:m3_Spacer_Hole_hex, F.Cu at (198.9, 129.1)
- added SW57: SW_Push, Salicylic-acid3_kbd_SW:CherryMX_Solder_1u, F.Cu at (103.6, 116.8)
- added SW64: SW_Push, Salicylic-acid3_kbd_SW:CherryMX_Solder_1u, F.Cu at (267.4, 116.8)
- moved D1 0.56 mm to (47.1, 45.7)
- renumbered D57 to D58, D58 to D59, D59 to D60, D60 to D61, D61 to D62, D62 to D63, SW57 to SW58, SW58 to SW59, SW59 to SW60, SW60 to SW61, SW61 to SW62, SW62 to SW63
Routing:
- net GND: track 204.0 -> 223.6 mm, vias 5 -> 7
- net Col2: track 126.0 -> 110.7 mm
- net Net-(D64-A): track 0.00 -> 10.2 mm, vias 0 -> 1
- net Net-(D57-A): track 0.00 -> 10.2 mm, vias 0 -> 1
- net Col1: track 106.8 -> 96.9 mm, vias 3 -> 1
- net VDD: track 170.8 -> 176.3 mm
- net Col10: track 105.7 -> 111.1 mm
- net VCC: track 189.4 -> 194.1 mm, vias 1 -> 3
- net Col5: track 140.3 -> 136.2 mm, vias 4 -> 3
- net DataRight: track 184.3 -> 181.6 mm
- net Col7: track 182.6 -> 185.0 mm
- net Col13: track 116.9 -> 119.2 mm, vias 3 -> 2
- net Col8: track 165.2 -> 167.4 mm
- net Row8: track 160.1 -> 157.8 mm
- net Row2: track 143.6 -> 145.3 mm
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Other:
- board size 301.3 x 112 mm -> 301.3 x 109 mm

Commit message: fix PCB Edge.Cuts
Parts:
- removed REF** (x10): m3_Spacer_Hole_hex, keyboard_parts:m3_Spacer_Hole_hex
- removed REF**: USB_type-C_dip_module_AE-USB2.0-TYPE-C, keyboard_parts:USB_type-C_dip_module_AE-USB2.0-TYPE-C
Connections:
- SW11 pad 1: Col10 -> Net-(SW11-Pad1)
- SW12 pad 1: Col11 -> Net-(SW12-Pad1)
- SW13 pad 1: Col12 -> Net-(SW13-Pad1)
- SW14 pad 1: Col13 -> Net-(SW14-Pad1)
- SW25 pad 1: Col10 -> Net-(SW11-Pad1)
- SW26 pad 1: Col11 -> Net-(SW12-Pad1)
- SW27 pad 1: Col12 -> Net-(SW13-Pad1)
- SW28 pad 1: Col13 -> Net-(SW14-Pad1)
- SW39 pad 1: Col10 -> Net-(SW11-Pad1)
- SW40 pad 1: Col11 -> Net-(SW12-Pad1)
- SW41 pad 1: Col12 -> Net-(SW13-Pad1)
- SW42 pad 1: Col13 -> Net-(SW14-Pad1)
- SW53 pad 1: Col10 -> Net-(SW11-Pad1)
- SW54 pad 1: Col11 -> Net-(SW12-Pad1)
- SW55 pad 1: Col12 -> Net-(SW13-Pad1)
- SW56 pad 1: Col13 -> Net-(SW14-Pad1)
- SW64 pad 1: Col10 -> Net-(SW11-Pad1)
Routing:
- net GND: track 223.6 -> 228.1 mm
Other:
- board size 301.3 x 109 mm -> 309.8 x 111.2 mm

Commit message: GNDを塗りつぶし
Parts:
- added REF**: USB_type-C_dip_module_AE-USB2.0-TYPE-C, keyboard_parts:USB_type-C_dip_module_AE-USB2.0-TYPE-C, F.Cu at (103.5, 22.9)
Connections:
- SW11 pad 1: Net-(SW11-Pad1) -> Col10
- SW12 pad 1: Net-(SW12-Pad1) -> Col11
- SW13 pad 1: Net-(SW13-Pad1) -> Col12
- SW14 pad 1: Net-(SW14-Pad1) -> Col13
- SW25 pad 1: Net-(SW11-Pad1) -> Col10
- SW26 pad 1: Net-(SW12-Pad1) -> Col11
- SW27 pad 1: Net-(SW13-Pad1) -> Col12
- SW28 pad 1: Net-(SW14-Pad1) -> Col13
- SW39 pad 1: Net-(SW11-Pad1) -> Col10
- SW40 pad 1: Net-(SW12-Pad1) -> Col11
- SW41 pad 1: Net-(SW13-Pad1) -> Col12
- SW42 pad 1: Net-(SW14-Pad1) -> Col13
- SW53 pad 1: Net-(SW11-Pad1) -> Col10
- SW54 pad 1: Net-(SW12-Pad1) -> Col11
- SW55 pad 1: Net-(SW13-Pad1) -> Col12
- SW56 pad 1: Net-(SW14-Pad1) -> Col13
- SW64 pad 1: Net-(SW11-Pad1) -> Col10
Routing:
- net Col13: track 119.2 -> 123.4 mm, vias 2 -> 3
- net Col10: track 111.1 -> 112.8 mm
- added copper zone on B.Cu, net GND
- added copper zone on F.Cu, net GND

Commit message: print version 0.1
Routing:
- added copper zone on B.Cu, net GNDA
- added copper zone on F.Cu, net GNDA
Other:
- board text added: "11111 ver.1 left hand"
- board text added: "11111 ver.1 right hand"
Changed lines of the file:
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@@
     (pad_to_mask_clearance 0)
     (pcbplotparams
-      (layerselection 0x00010fc_ffffffff)
+      (layerselection 0x00010f0_ffffffff)
       (plot_on_all_layers_selection 0x0000000_00000000)
       (disableapertmacros false)
@@
       (outputformat 1)
       (mirror false)
-      (drillshape 1)
+      (drillshape 0)
       (scaleselection 1)
-      (outputdirectory "")
+      (outputdirectory "../gerbers/v0.1/PCB/")
     )
   )
@@
   (gr_line (start 33.02 22.86) (end 175.303949 22.856051)
     (stroke (width 0.1) (type default)) (layer "Edge.Cuts"))
+  (gr_text "11111 ver.1\nleft hand" (at 170.18 30.28) (layer "B.SilkS")
+    (effects (font (size 1.5 1.5) (thickness 0.3) bold) (justify left bottom mirror))
+  )
+  (gr_text "11111 ver.1\nright hand" (at 335.28 29.88) (layer "B.SilkS")
+    (effects (font (size 1.5 1.5) (thickness 0.3) bold) (justify left bottom mirror))
+  )
   (segment (start 74.23 103.57) (end 76.2 101.6) (width 0.25) (layer "F.Cu") (net 1))
   (segment (start 76.2 101.6) (end 76.2 49.22) (width 0.25) (layer "F.Cu") (net 1))
@@
   (segment (start 81.025128 120.204872) (end 79.31 121.92) (width 0.25) (layer "F.Cu") (net 84))
   (segment (start 114.3 114.3) (end 111.76 116.84) (width 0.25) (layer "F.Cu") (net 84))
-  (segment (start 111.76 116.84) (end 111.76 117.8) (width 0.25) (layer "F.Cu") (net 84))
   (segment (start 118.8 38.095) (end 118.8 114.185) (width 0.25) (layer "F.Cu") (net 84))
   (segment (start 111.76 117.8) (end 109.22 120.34) (width 0.25) (layer "F.Cu") (net 84))
+  (segment (start 111.76 116.84) (end 111.76 117.8) (width 0.25) (layer "F.Cu") (net 84))
   (segment (start 118.8 114.185) (end 118.745 114.24) (width 0.25) (layer "F.Cu") (net 84))
   (segment (start 118.745 38.04) (end 118.8 38.095) (width 0.25) (layer "F.Cu") (net 84))
@@
   (segment (start 269.995 121.88) (end 269.975 121.86) (width 0.25) (layer "F.Cu") (net 132))
   (via (at 269.995 121.88) (size 0.8) (drill 0.4) (layers "F.Cu" "B.Cu") (net 132))
-  (zone (net 74) (net_name "GND") (layers "F&B.Cu") (hatch edge 0.5)
+  (zone (net 113) (net_name "GNDA") (layers "F&B.Cu") (hatch edge 0.5)
     (connect_pads (clearance 0.508))
     (min_thickness 0.25) (filled_areas_thickness no)
-    (fill (thermal_gap 0.5) (thermal_bridge_width 0.5))
+    (fill yes (thermal_gap 0.5) (thermal_bridge_width 0.5))
     (polygon
       (pts
@@
     (connect_pads (clearance 0.508))
     (min_thickness 0.25) (filled_areas_thickness no)
-    (fill (thermal_gap 0.5) (thermal_bridge_width 0.5))
+    (fill yes (thermal_gap 0.5) (thermal_bridge_width 0.5))
     (polygon
       (pts
