File: blueprints/pcb/11111_pcb.kicad_pcb (KiCad board)
At the start: 2 copper layers, 298.5 x 111.2 mm, 139 parts, among them J1 TRRS_MJ-4PP-9, J2 TRRS_MJ-4PP-9, SW1 SW_Push, SW10 SW_Push, SW11 SW_Push, SW12 SW_Push, SW13 SW_Push, SW14 SW_Push, SW15 SW_Push, SW16 SW_Push, SW17 SW_Push, SW18 SW_Push, SW19 SW_Push, SW2 SW_Push, SW20 SW_Push, SW21 SW_Push, SW22 SW_Push, SW23 SW_Push, SW24 SW_Push, SW25 SW_Push, SW26 SW_Push, SW27 SW_Push, SW28 SW_Push, SW29 SW_Push, SW3 SW_Push, SW30 SW_Push, SW31 SW_Push, SW32 SW_Push, SW33 SW_Push, SW34 SW_Push, SW35 SW_Push, SW36 SW_Push, SW37 SW_Push, SW38 SW_Push, SW39 SW_Push, SW4 SW_Push, SW40 SW_Push, SW41 SW_Push, SW42 SW_Push, SW43 SW_Push, SW44 SW_Push, SW45 SW_Push, SW46 SW_Push, SW47 SW_Push, SW48 SW_Push, SW49 SW_Push, SW5 SW_Push, SW50 SW_Push, SW51 SW_Push, SW52 SW_Push, SW53 SW_Push, SW54 SW_Push, SW55 SW_Push, SW56 SW_Push, SW57 SW_Push, SW58 SW_Push, SW59 SW_Push, SW6 SW_Push, SW60 SW_Push, SW61 SW_Push, SW62 SW_Push, SW63 SW_Push, SW64 SW_Push, SW7 SW_Push, SW8 SW_Push, SW9 SW_Push, U1 Pico, U2 Pico

Commit message: narrow right PCB
Parts:
- removed the REF** at (186.4, 25.7)
- removed the REF** at (322.0, 25.7)
- removed the REF** at (186.4, 126.7)
- removed the REF** at (265.5, 126.7)
- moved J2 46.4 mm to (209.2, 26.6), turned to 0 degrees
- moved D54 11.9 mm to (264.2, 94.8), turned to 90 degrees
- moved D56 11.6 mm to (302.5, 94.8), turned to 90 degrees
- moved D55 11.6 mm to (283.4, 94.9), turned to 90 degrees
- moved J1 11.0 mm to (141.4, 26.6), turned to 0 degrees
- moved REF** 10.9 mm to (128.1, 20.3)
- moved U2 2.48 mm to (295.5, 111.6)
- moved D44 1.20 mm to (66.0, 94.7)
Routing:
- net GND: track 0.00 -> 251.6 mm, vias 0 -> 7
- net VCC: track 0.00 -> 192.0 mm, vias 0 -> 2
- net DataLeft: track 0.00 -> 179.9 mm, vias 0 -> 2
- net GNDA: track 237.3 -> 316.7 mm, vias 3 -> 9
- net Row3: track 63.2 -> 137.7 mm, vias 0 -> 2
- net Row8: track 157.8 -> 138.7 mm, vias 4 -> 2
- net DataRight: track 181.6 -> 194.2 mm, vias 3 -> 2
- net Row5: track 212.5 -> 224.0 mm
- net Row0: track 179.5 -> 190.7 mm, vias 1 -> 2
- net Col7: track 185.0 -> 195.1 mm
- net Net-(D43-A): track 0.00 -> 8.12 mm
- net Net-(D45-A): track 0.00 -> 8.12 mm
- net Net-(D44-A): track 0.00 -> 6.92 mm
- net VDD: track 176.3 -> 183.1 mm, vias 3 -> 2
- net Col11: track 80.3 -> 74.3 mm, vias 2 -> 1
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Other:
- board size 298.5 x 111.2 mm -> 292.4 x 103.6 mm
- board text added: "11111 ver.2 left hand"
- board text added: "11111 ver.2 right hand"
- board text removed: "11111 ver.1 left hand"
- board text removed: "11111 ver.1 right hand"

Commit message: modify PCB
Parts:
- moved J2 0.10 mm to (209.3, 26.6)
Routing:
- net GND: track 251.6 -> 248.9 mm
Other:
- outline, holes or cut-outs redrawn

Commit message: version3
Parts:
- removed the REF** at (128.1, 20.3)
- removed U1, U2: Pico, Raspberry-pi-pico:RPi_Pico_SMD_TH
- added A1: RP2040-Zero, RP2040-zero:RP2040-Zero_through_hole_omit, B.Cu at (132.6, 32.7)
- added A2: RP2040-Zero, RP2040-zero:RP2040-Zero_through_hole_omit, B.Cu at (218.2, 32.7)
- moved D9 10.4 mm to (207.2, 41.7), turned to 90 degrees
- moved D6 9.06 mm to (143.5, 40.9), turned to 90 degrees
- moved J1 3.38 mm to (144.8, 26.6)
- moved J2 3.25 mm to (206.1, 26.6)
- moved SW43 0.10 mm to (38.7, 95.2)
- moved SW44 0.10 mm to (57.7, 95.2)
- moved SW45 0.10 mm to (76.8, 95.2)
- moved SW46 0.08 mm to (95.9, 95.2)
- moved SW47 0.08 mm to (114.9, 95.2)
- moved SW48 0.08 mm to (134.0, 95.2)
Routing:
- net GNDA: track 316.7 -> 29.0 mm, vias 9 -> 0
- net GND: track 248.9 -> 3.03 mm, vias 7 -> 0
- net VCC: track 192.0 -> 12.3 mm, vias 2 -> 0
- net DataLeft: track 179.9 -> 14.5 mm, vias 2 -> 0
- net DataRight: track 194.1 -> 32.1 mm, vias 2 -> 1
- net VDD: track 183.0 -> 28.4 mm, vias 2 -> 1
- net Row5: track 224.0 -> 128.0 mm, vias 2 -> 0
- net Col7: track 195.0 -> 102.2 mm, vias 3 -> 1
- net Col8: track 170.3 -> 90.6 mm, vias 4 -> 0
- net Col0: track 103.6 -> 172.0 mm, vias 2 -> 1
- net Col12: track 78.6 -> 141.9 mm, vias 1 -> 2
- net Row9: track 81.0 -> 142.2 mm, vias 0 -> 3
- net Col6: track 156.8 -> 99.1 mm, vias 1 -> 2
- net Row0: track 190.7 -> 134.9 mm, vias 2 -> 0
- net Row4: track 87.5 -> 142.3 mm, vias 4 -> 1
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- added copper zone on B.Cu, net (none)
- added copper zone on F.Cu, net (none)
- removed copper zone on B.Cu, net GND
- removed copper zone on F.Cu, net GND
- removed copper zone on B.Cu, net GNDA
- removed copper zone on F.Cu, net GNDA
Other:
- outline, holes or cut-outs redrawn
- board text added: "11111 ver.3 left hand"
- board text added: "11111 ver.3 right hand"
- board text removed: "11111 ver.2 left hand"
- board text removed: "11111 ver.2 right hand"
