File: blueprints/pcb/pcb.kicad_pcb (KiCad board)
At the start: 2 copper layers, 292.4 x 103.6 mm, 134 parts, among them J1 TRRS_MJ-4PP-9, J2 TRRS_MJ-4PP-9, SW1 SW_Push, SW10 SW_Push, SW11 SW_Push, SW12 SW_Push, SW13 SW_Push, SW14 SW_Push, SW15 SW_Push, SW16 SW_Push, SW17 SW_Push, SW18 SW_Push, SW19 SW_Push, SW2 SW_Push, SW20 SW_Push, SW21 SW_Push, SW22 SW_Push, SW23 SW_Push, SW24 SW_Push, SW25 SW_Push, SW26 SW_Push, SW27 SW_Push, SW28 SW_Push, SW29 SW_Push, SW3 SW_Push, SW30 SW_Push, SW31 SW_Push, SW32 SW_Push, SW33 SW_Push, SW34 SW_Push, SW35 SW_Push, SW36 SW_Push, SW37 SW_Push, SW38 SW_Push, SW39 SW_Push, SW4 SW_Push, SW40 SW_Push, SW41 SW_Push, SW42 SW_Push, SW43 SW_Push, SW44 SW_Push, SW45 SW_Push, SW46 SW_Push, SW47 SW_Push, SW48 SW_Push, SW49 SW_Push, SW5 SW_Push, SW50 SW_Push, SW51 SW_Push, SW52 SW_Push, SW53 SW_Push, SW54 SW_Push, SW55 SW_Push, SW56 SW_Push, SW57 SW_Push, SW58 SW_Push, SW59 SW_Push, SW6 SW_Push, SW60 SW_Push, SW61 SW_Push, SW62 SW_Push, SW63 SW_Push, SW64 SW_Push, SW7 SW_Push, SW8 SW_Push, SW9 SW_Push

Commit message: fix silk print
Other:
- board text added: "64 ver.3 left hand"
- board text added: "64 ver.3 right hand"
- board text removed: "11111 ver.3 left hand"
- board text removed: "11111 ver.3 right hand"
Changed lines of the file:
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@@
   (gr_line (start 123.5118 20.32) (end 147.9296 20.32)
     (stroke (width 0.1) (type default)) (layer "Edge.Cuts"))
-  (gr_text "11111 ver.3\nleft hand" (at 60.96 104.394) (layer "B.SilkS")
+  (gr_text "64 ver.3\nleft hand" (at 60.96 104.394) (layer "B.SilkS")
     (effects (font (size 1.5 1.5) (thickness 0.3) bold) (justify left bottom mirror))
   )
-  (gr_text "11111 ver.3\nright hand" (at 304.8 104.14) (layer "B.SilkS")
+  (gr_text "64 ver.3\nright hand" (at 304.8 104.14) (layer "B.SilkS")
     (effects (font (size 1.5 1.5) (thickness 0.3) bold) (justify left bottom mirror))
   )
