File: blueprints/plates/11111_plates.kicad_pcb (KiCad board)
At the start: 2 copper layers, 306.4 x 228.2 mm, 84 parts, among them SW1 SW_Push, SW10 SW_Push, SW11 SW_Push, SW12 SW_Push, SW13 SW_Push, SW14 SW_Push, SW15 SW_Push, SW16 SW_Push, SW17 SW_Push, SW18 SW_Push, SW19 SW_Push, SW2 SW_Push, SW20 SW_Push, SW21 SW_Push, SW22 SW_Push, SW23 SW_Push, SW24 SW_Push, SW25 SW_Push, SW26 SW_Push, SW27 SW_Push, SW28 SW_Push, SW29 SW_Push, SW3 SW_Push, SW30 SW_Push, SW31 SW_Push, SW32 SW_Push, SW33 SW_Push, SW34 SW_Push, SW35 SW_Push, SW36 SW_Push, SW37 SW_Push, SW38 SW_Push, SW39 SW_Push, SW4 SW_Push, SW40 SW_Push, SW41 SW_Push, SW42 SW_Push, SW43 SW_Push, SW44 SW_Push, SW45 SW_Push, SW46 SW_Push, SW47 SW_Push, SW48 SW_Push, SW49 SW_Push, SW5 SW_Push, SW50 SW_Push, SW51 SW_Push, SW52 SW_Push, SW53 SW_Push, SW54 SW_Push, SW55 SW_Push, SW56 SW_Push, SW57 SW_Push, SW58 SW_Push, SW59 SW_Push, SW6 SW_Push, SW60 SW_Push, SW61 SW_Push, SW62 SW_Push, SW63 SW_Push, SW64 SW_Push, SW7 SW_Push, SW8 SW_Push, SW9 SW_Push

Commit message: modify plate
Parts:
- moved REF** 3.75 mm to (92.5, 128.5)
- moved REF** 3.75 mm to (171.5, 128.5)
- moved SW29 3.75 mm to (45.9, 78.0)
- moved SW30 3.75 mm to (64.8, 78.0)
- moved SW31 3.75 mm to (84.0, 78.0)
- moved SW32 3.75 mm to (103.0, 78.0)
- moved SW33 3.75 mm to (122.1, 78.0)
- moved SW34 3.75 mm to (141.1, 78.0)
- moved SW35 3.75 mm to (160.2, 78.0)
- moved SW43 3.75 mm to (45.9, 97.2)
- moved SW44 3.75 mm to (64.8, 97.2)
- moved SW45 3.75 mm to (84.0, 97.2)
- moved SW46 3.75 mm to (103.0, 97.2)
- moved SW47 3.75 mm to (122.1, 97.2)
- moved SW48 3.75 mm to (141.1, 97.2)
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Other:
- board size 306.4 x 228.2 mm -> 306.1 x 228.1 mm
- board text added: "11111 ver.1"
- board text removed: "11111 ver.1 left hand"
- board text removed: "11111 ver.1 right hand"

Commit message: modify PCB and plates
Other:
- board text added: "deprecated.(same for both hands) use left only."
Changed lines of the file:
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@@
     (effects (font (size 1.5 1.5) (thickness 0.3) bold) (justify left bottom))
   )
+  (gr_text "deprecated.(same for both hands)\nuse left only." (at 281.94 116.84) (layer "Eco1.User")
+    (effects (font (size 2 2) (thickness 0.15)) (justify left bottom))
+  )
+  (gr_text "deprecated.(same for both hands)\nuse left only." (at 281.94 154.94) (layer "Eco1.User")
+    (effects (font (size 2 2) (thickness 0.15)) (justify left bottom))
+  )
 )

Commit message: fix
Parts:
- moved REF** 7.36 mm to (85.4, 126.6)
- moved REF** 7.36 mm to (164.4, 126.6)
- moved SW31 7.36 mm to (76.8, 76.1)
- moved SW33 7.36 mm to (114.9, 76.1)
- moved SW35 7.36 mm to (153.0, 76.1)
- moved SW45 7.36 mm to (76.8, 95.3)
- moved SW47 7.36 mm to (114.9, 95.3)
- moved SW17 7.36 mm to (76.8, 57.1)
- moved SW19 7.36 mm to (114.9, 57.1)
- moved SW21 7.36 mm to (153.0, 57.1)
- moved SW3 7.36 mm to (76.8, 38.0)
- moved SW5 7.36 mm to (114.9, 38.0)
- moved SW7 7.36 mm to (153.0, 38.0)
- moved REF** 7.36 mm to (164.4, 25.7)
- moved REF** 7.36 mm to (164.4, 240.9)
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Other:
- board size 306.1 x 228.1 mm -> 313.2 x 227.3 mm

Commit message: update
Parts:
- SW1, SW10, SW11, SW12, SW13, SW14, SW15, SW16, SW17, SW18, SW19, SW2, SW20, SW21, SW22, SW23, SW24, SW25, SW26, SW27, SW28, SW29, SW3, SW30, SW31, SW32, SW33, SW34, SW35, SW36, SW37, SW38, SW39, SW4, SW40, SW41, SW42, SW43, SW44, SW45, SW46, SW47, SW48, SW49, SW5, SW50, SW51, SW52, SW53, SW54, SW55, SW56, SW57, SW58, SW59, SW6, SW60, SW61, SW62, SW63, SW64, SW7, SW8, SW9: footprint foostan:SW_Hole -> Salicylic-acid3_kbd_SW_Hole:SW_Hole_TH_1u
