File: blueprints/plates/11111_plates.kicad_pcb (KiCad board)
At the start: 2 copper layers, 313.2 x 227.3 mm, 84 parts, among them SW1 SW_Push, SW10 SW_Push, SW11 SW_Push, SW12 SW_Push, SW13 SW_Push, SW14 SW_Push, SW15 SW_Push, SW16 SW_Push, SW17 SW_Push, SW18 SW_Push, SW19 SW_Push, SW2 SW_Push, SW20 SW_Push, SW21 SW_Push, SW22 SW_Push, SW23 SW_Push, SW24 SW_Push, SW25 SW_Push, SW26 SW_Push, SW27 SW_Push, SW28 SW_Push, SW29 SW_Push, SW3 SW_Push, SW30 SW_Push, SW31 SW_Push, SW32 SW_Push, SW33 SW_Push, SW34 SW_Push, SW35 SW_Push, SW36 SW_Push, SW37 SW_Push, SW38 SW_Push, SW39 SW_Push, SW4 SW_Push, SW40 SW_Push, SW41 SW_Push, SW42 SW_Push, SW43 SW_Push, SW44 SW_Push, SW45 SW_Push, SW46 SW_Push, SW47 SW_Push, SW48 SW_Push, SW49 SW_Push, SW5 SW_Push, SW50 SW_Push, SW51 SW_Push, SW52 SW_Push, SW53 SW_Push, SW54 SW_Push, SW55 SW_Push, SW56 SW_Push, SW57 SW_Push, SW58 SW_Push, SW59 SW_Push, SW6 SW_Push, SW60 SW_Push, SW61 SW_Push, SW62 SW_Push, SW63 SW_Push, SW64 SW_Push, SW7 SW_Push, SW8 SW_Push, SW9 SW_Push

Commit message: print 'ver.2' on plates
Other:
- board text added: "11111 ver.2"
- board text removed: "11111 ver.1"
Changed lines of the file:
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@@
     (pad "1" thru_hole oval (at 6.95 0) (size 2 15.9) (drill oval 0.3 14.2) (layers "*.Cu" "*.Mask"))
   )
-  (gr_rect (start 29.2 28.4) (end 162.64 123.8)
+  (gr_rect (start 29.2 28.5) (end 162.6 123.75)
     (stroke (width 0.15) (type default)) (fill none) (layer "Cmts.User"))
   (gr_arc (start 170.223949 128.836051) (mid 169.479985 130.632087) (end 167.683949 131.376051)
@@
   (gr_line (start 25.4 20.316051) (end 167.683949 20.312102)
     (stroke (width 0.1) (type default)) (layer "Edge.Cuts"))
-  (gr_text "11111 ver.1" (at 27.94 231.88) (layer "F.SilkS")
+  (gr_text "11111 ver.2" (at 27.94 231.88) (layer "F.SilkS")
     (effects (font (size 1.5 1.5) (thickness 0.3) bold) (justify left bottom))
   )
-  (gr_text "11111 ver.1" (at 27.94 120.12) (layer "F.SilkS")
+  (gr_text "11111 ver.2" (at 27.94 120.12) (layer "F.SilkS")
     (effects (font (size 1.5 1.5) (thickness 0.3) bold) (justify left bottom))
   )

Commit message: export top plate step file from KiCad
Parts:
- removed the REF** at (310.0, 200.9)
- removed the REF** at (194.7, 125.8)
- removed the REF** at (194.7, 24.7)
- removed the REF** at (329.6, 140.9)
- removed the REF** at (194.0, 140.8)
- removed the REF** at (273.7, 125.7)
- removed the REF** at (48.3, 200.1)
- removed the REF** at (310.8, 84.8)
- removed the REF** at (272.9, 241.8)
- removed the REF** at (330.3, 24.8)
- removed the REF** at (194.0, 241.9)
- removed the REF** at (48.3, 85.8)
- removed SW10, SW11, SW12, SW13, SW14, SW22, SW23, SW24, SW25, SW26, SW27, SW28, SW36, SW37, SW38, SW39, SW40, SW41, SW42, SW50, SW51, SW52, SW53, SW54, SW55, SW56, SW61, SW62, SW63, SW64, SW8, SW9: SW_Push, Salicylic-acid3_kbd_SW_Hole:SW_Hole_TH_1u
- moved REF** 194.6 mm to (321.9, 126.6)
- moved REF** 194.6 mm to (321.9, 25.7)
- moved REF** 194.6 mm to (186.2, 25.7)
- moved REF** 152.4 mm to (186.2, 126.6)
- moved REF** 56.6 mm to (28.8, 126.6)
Other:
- board size 313.2 x 227.3 mm -> 304.8 x 111.1 mm
- board text added: "11111 ver.3"
- board text removed: "11111 ver.2"
- board text removed: "deprecated.(same for both hands) use left only."

Commit message: update silk print text
Other:
- board text added: "64 ver.3"
- board text removed: "11111 ver.3"
Changed lines of the file:
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@@
   (gr_line (start 25.4 20.316051) (end 167.683949 20.312102)
     (stroke (width 0.1) (type default)) (layer "Edge.Cuts"))
-  (gr_text "11111 ver.3" (at 185.398025 117.585923) (layer "F.SilkS")
+  (gr_text "64 ver.3" (at 185.398025 117.585923) (layer "F.SilkS")
     (effects (font (size 1.5 1.5) (thickness 0.3) bold) (justify left bottom))
   )
-  (gr_text "11111 ver.3" (at 27.94 120.12) (layer "F.SilkS")
+  (gr_text "64 ver.3" (at 27.94 120.12) (layer "F.SilkS")
     (effects (font (size 1.5 1.5) (thickness 0.3) bold) (justify left bottom))
   )
